Commit message: Updating bundle to console version

File: simulation/aws-robomaker-sample-application-deepracer/simulation_ws/src/deepracer_simulation/urdf/racecar.xacro (robot description, xacro)
@@ -167,5 +167,5 @@
   </link>
   <joint name="zed_camera_joint" type="fixed">
-    <origin xyz="0.20 0 0.10" rpy="0 0.2731415 0"/>
+    <origin xyz="0.20 0 0.134" rpy="0 0.261799 0"/>
     <parent link="chassis"/>
     <child link="zed_camera_link"/>
